Commit message: 右アームにカメラを追加

File: urdf/right_gemini_335_336.urdf.xacro (robot description, xacro)
@@ -6,5 +6,6 @@
 <robot xmlns:xacro="http://ros.org/wiki/xacro" name="gemini_335_336">
     <xacro:property name="mesh_path" value="package://sciurus17_description/meshes/gemini335_336/" />
-    <link name="camera_link">
+    <xacro:property name="prefix" value="right_"/>
+    <link name="${prefix}camera_link">
         <inertial>
             <origin xyz="0.00277269933215555 -1.06084680351007E-05 0.012801025085723" rpy="0 0 0" />
@@ -30,5 +31,5 @@
         </collision>
     </link>
-    <link name="camera_bottom_screw_frame">
+    <link name="${prefix}camera_bottom_screw_frame">
         <inertial>
             <origin xyz="0.00255168206289301 -0.00123934714960528 0.0118889875786098" rpy="0 0 0" />
@@ -54,11 +55,11 @@
         </collision> -->
     </link>
-    <joint name="camera_bottom_screw_frame_joint" type="fixed">
+    <joint name="${prefix}camera_bottom_screw_frame_joint" type="fixed">
         <origin xyz="0 0 0" rpy="0 0 0" />
-        <parent link="camera_link" />
-        <child link="camera_bottom_screw_frame" />
-        <axis xyz="0 0 0" />
-    </joint>
-    <link name="camera_infra_1_frame">
+        <parent link="${prefix}camera_link" />
+        <child link="${prefix}camera_bottom_screw_frame" />
+        <axis xyz="0 0 0" />
+    </joint>
+    <link name="${prefix}camera_infra_1_frame">
         <inertial>
             <origin xyz="-0.00158020887627678 -1.52683853303637E-08 -1.4860800305164E-07"
@@ -85,11 +86,11 @@
         </collision> -->
     </link>
-    <joint name="camera_infra_1_joint" type="fixed">
+    <joint name="${prefix}camera_infra_1_joint" type="fixed">
         <origin xyz="0.01587 -0.025 0.0125" rpy="0 0 0" />
-        <parent link="camera_bottom_screw_frame" />
-        <child link="camera_infra_1_frame" />
-        <axis xyz="0 0 0" />
-    </joint>
-    <link name="camera_infra_1_optical_frame">
+        <parent link="${prefix}camera_bottom_screw_frame" />
+        <child link="${prefix}camera_infra_1_frame" />
+        <axis xyz="0 0 0" />
+    </joint>
+    <link name="${prefix}camera_infra_1_optical_frame">
         <inertial>
             <origin xyz="1.52683853338331E-08 1.48608003051636E-07 -0.00158020887627678" rpy="0 0 0" />
@@ -115,11 +116,11 @@
         </collision> -->
     </link>
-    <joint name="camera_infra_1_optical_joint" type="fixed">
+    <joint name="${prefix}camera_infra_1_optical_joint" type="fixed">
         <origin xyz="0.01587 -0.025 0.0125" rpy="-1.5707963267949 0 -1.5707963267949" />
-        <parent link="camera_bottom_screw_frame" />
-        <child link="camera_infra_1_optical_frame" />
-        <axis xyz="0 0 0" />
-    </joint>
-    <link name="camera_infra2_frame">
+        <parent link="${prefix}camera_bottom_screw_frame" />
+        <child link="${prefix}camera_infra_1_optical_frame" />
+        <axis xyz="0 0 0" />
+    </joint>
+    <link name="${prefix}camera_infra2_frame">
         <inertial>
             <origin xyz="-0.00158020887627678 -1.52683853303637E-08 -1.48608003050581E-07"
@@ -146,11 +147,11 @@
         </collision> -->
     </link>
-    <joint name="camera_infra2_joint" type="fixed">
+    <joint name="${prefix}camera_infra2_joint" type="fixed">
         <origin xyz="0.01587 0.025 0.0125" rpy="0 0 0" />
-        <parent link="camera_bottom_screw_frame" />
-        <child link="camera_infra2_frame" />
-        <axis xyz="0 0 0" />
-    </joint>
-    <link name="camera_infra2_optical_frame">
+        <parent link="${prefix}camera_bottom_screw_frame" />
+        <child link="${prefix}camera_infra2_frame" />
+        <axis xyz="0 0 0" />
+    </joint>
+    <link name="${prefix}camera_infra2_optical_frame">
         <inertial>
             <origin xyz="1.52683853268942E-08 1.4860800305058E-07 -0.00158020887627678" rpy="0 0 0" />
@@ -176,11 +177,11 @@
         </collision> -->
     </link>
-    <joint name="camera_infra2_optical_joint" type="fixed">
+    <joint name="${prefix}camera_infra2_optical_joint" type="fixed">
         <origin xyz="0.01587 0.025 0.0125" rpy="-1.5707963267949 0 -1.5707963267949" />
-        <parent link="camera_bottom_screw_frame" />
-        <child link="camera_infra2_optical_frame" />
-        <axis xyz="0 0 0" />
-    </joint>
-    <link name="camera_color_frame">
+        <parent link="${prefix}camera_bottom_screw_frame" />
+        <child link="${prefix}camera_infra2_optical_frame" />
+        <axis xyz="0 0 0" />
+    </joint>
+    <link name="${prefix}camera_color_frame">
         <inertial>
             <origin xyz="-0.00177079701156752 -2.20101367029782E-07 2.09893364599916E-07"
@@ -207,11 +208,11 @@
         </collision> -->
     </link>
-    <joint name="camera_color_joint" type="fixed">
+    <joint name="${prefix}camera_color_joint" type="fixed">
         <origin xyz="0.017533 0.010995 0.012505" rpy="0 0 0" />
-        <parent link="camera_bottom_screw_frame" />
-        <child link="camera_color_frame" />
-        <axis xyz="0 0 0" />
-    </joint>
-    <link name="camera_color_optical_frame">
+        <parent link="${prefix}camera_bottom_screw_frame" />
+        <child link="${prefix}camera_color_frame" />
+        <axis xyz="0 0 0" />
+    </joint>
+    <link name="${prefix}camera_color_optical_frame">
         <inertial>
             <origin xyz="2.20101367029782E-07 -2.09893364599916E-07 -0.00177079701156752"
@@ -238,11 +239,11 @@
         </collision> -->
     </link>
-    <joint name="camera_color_optical_joint" type="fixed">
+    <joint name="${prefix}camera_color_optical_joint" type="fixed">
         <origin xyz="0.017533 0.010995 0.012505" rpy="-1.5707963267949 0 -1.5707963267949" />
-        <parent link="camera_bottom_screw_frame" />
-        <child link="camera_color_optical_frame" />
-        <axis xyz="0 0 0" />
-    </joint>
-    <link name="camera_depth_frame">
+        <parent link="${prefix}camera_bottom_screw_frame" />
+        <child link="${prefix}camera_color_optical_frame" />
+        <axis xyz="0 0 0" />
+    </joint>
+    <link name="${prefix}camera_depth_frame">
         <inertial>
             <origin xyz="-0.00158020887627678 -1.52683853338331E-08 -1.48608003051662E-07"
@@ -269,11 +270,11 @@
         </collision> -->
     </link>
-    <joint name="camera_depth_joint" type="fixed">
+    <joint name="${prefix}camera_depth_joint" type="fixed">
         <origin xyz="0.01587 -0.025 0.0125" rpy="0 0 0" />
-        <parent link="camera_bottom_screw_frame" />
-        <child link="camera_depth_frame" />
-        <axis xyz="0 0 0" />
-    </joint>
-    <link name="camera_depth_optical_frame">
+        <parent link="${prefix}camera_bottom_screw_frame" />
+        <child link="${prefix}camera_depth_frame" />
+        <axis xyz="0 0 0" />
+    </joint>
+    <link name="${prefix}camera_depth_optical_frame">
         <inertial>
             <origin xyz="1.52683853338331E-08 1.4860800305165E-07 -0.00158020887627678" rpy="0 0 0" />
@@ -298,8 +299,8 @@
         </collision> -->
     </link>
-    <joint name="camera_depth_optical_joint" type="fixed">
+    <joint name="${prefix}camera_depth_optical_joint" type="fixed">
         <origin xyz="0.01587 -0.025 0.0125" rpy="-1.5707963267949 0 -1.5707963267949" />
-        <parent link="camera_bottom_screw_frame" />
-        <child link="camera_depth_optical_frame" />
+        <parent link="${prefix}camera_bottom_screw_frame" />
+        <child link="${prefix}camera_depth_optical_frame" />
         <axis xyz="0 0 0" />
     </joint>

File: urdf/sciurus17.urdf.xacro (robot description, xacro)
@@ -184,9 +184,9 @@
   <!-- 左アーム -->
   <!-- Gemini カメラの組み込み -->
-  <xacro:include filename="$(find sciurus17_description)/urdf/_gemini_335_336.urdf.xacro"/>
+  <xacro:include filename="$(find sciurus17_description)/urdf/left_gemini_335_336.urdf.xacro"/>
   <!-- 固定ジョイント -->
-  <joint name="gemini_camera_mount_joint" type="fixed">
+  <joint name="left_gemini_camera_mount_joint" type="fixed">
     <parent link="l_link7"/>
-    <child link="camera_link"/>
+    <child link="left_camera_link"/>
     <!-- 要調整：mm単位でのズレをxyz, 向きのずれをrpyで指定 -->
     <origin xyz="0.0 0.02 0.03" rpy="0 0 1.57"/>
@@ -194,11 +194,11 @@
   <!-- 右アーム -->
   <!-- Gemini カメラの組み込み -->
-  <!-- <xacro:include filename="$(find sciurus17_description)/urdf/gemini_335_336_camera.xacro"/> -->
+  <xacro:include filename="$(find sciurus17_description)/urdf/right_gemini_335_336.urdf.xacro"/>
   <!-- 固定ジョイント -->
-  <!-- <joint name="gemini_camera_mount_joint" type="fixed">
+  <joint name="right_gemini_camera_mount_joint" type="fixed">
     <parent link="r_link7"/>
-    <child link="camera_link"/> -->
+    <child link="right_camera_link"/>
     <!-- 要調整：mm単位でのズレをxyz, 向きのずれをrpyで指定 -->
-    <!-- <origin xyz="0.0 -0.032 -0.0191" rpy="-1.57 1.57 0.0"/>
-  </joint> -->
+    <origin xyz="0.0 -0.02 -0.03" rpy="3.14 0 -1.57"/>
+  </joint>
 </robot>
