Commit message: 左アームにカメラを追加

File: urdf/sciurus17.urdf.xacro (robot description, xacro)
@@ -182,3 +182,23 @@
     <link name="${NAME_HEAD_CAMERA_PREFIX}_color_optical_frame"/>
   </xacro:if>
+  <!-- 左アーム -->
+  <!-- Gemini カメラの組み込み -->
+  <xacro:include filename="$(find sciurus17_description)/urdf/_gemini_335_336.urdf.xacro"/>
+  <!-- 固定ジョイント -->
+  <joint name="gemini_camera_mount_joint" type="fixed">
+    <parent link="l_link7"/>
+    <child link="camera_link"/>
+    <!-- 要調整：mm単位でのズレをxyz, 向きのずれをrpyで指定 -->
+    <origin xyz="0.0 0.02 0.03" rpy="0 0 1.57"/>
+  </joint>
+  <!-- 右アーム -->
+  <!-- Gemini カメラの組み込み -->
+  <!-- <xacro:include filename="$(find sciurus17_description)/urdf/gemini_335_336_camera.xacro"/> -->
+  <!-- 固定ジョイント -->
+  <!-- <joint name="gemini_camera_mount_joint" type="fixed">
+    <parent link="r_link7"/>
+    <child link="camera_link"/> -->
+    <!-- 要調整：mm単位でのズレをxyz, 向きのずれをrpyで指定 -->
+    <!-- <origin xyz="0.0 -0.032 -0.0191" rpy="-1.57 1.57 0.0"/>
+  </joint> -->
 </robot>

Commit message: 衝突判定のため棚を追加

File: urdf/sciurus17.urdf.xacro (robot description, xacro)
@@ -202,3 +202,73 @@
     <origin xyz="0.0 -0.02 -0.03" rpy="3.14 0 -1.57"/>
   </joint>
+  <!-- 棚を追加し、衝突判定する -->
+  <!-- 1段目 -->
+  <link name="first_shelf">
+    <visual>
+      <origin xyz="0.0 0.0 0.0" rpy="0 0 0" />
+      <geometry>
+        <box size="0.95 0.454 0.0005" />
+      </geometry>
+      <material name="light_yellow">
+        <color rgba="01.0 1.0 0.7 1.0" />
+      </material>
+    </visual>
+    <collision>
+      <origin xyz="0.0 0.0 0.0" rpy="0 0 0" />
+      <geometry>
+        <box size="0.95 0.454 0.0005" />
+      </geometry>
+    </collision>
+  </link>
+  <joint name="first_shelf_joint" type="fixed">
+    <parent link="base_link"/>
+    <child link="first_shelf"/>
+    <origin xyz="0.0 -0.6 0.198" rpy="0 0 0"/>
+  </joint>
+  <!-- 2段目 -->
+  <link name="2nd_shelf">
+    <visual>
+      <origin xyz="0.0 0.0 0.0" rpy="0 0 0" />
+      <geometry>
+        <box size="0.95 0.454 0.0005" />
+      </geometry>
+      <material name="light_yellow">
+        <color rgba="01.0 1.0 0.7 1.0" />
+      </material>
+    </visual>
+    <collision>
+      <origin xyz="0.0 0.0 0.0" rpy="0 0 0" />
+      <geometry>
+        <box size="0.95 0.454 0.0005" />
+      </geometry>
+    </collision>
+  </link>
+  <joint name="2nd_shelf_joint" type="fixed">
+    <parent link="base_link"/>
+    <child link="2nd_shelf"/>
+    <origin xyz="0.0 -0.6 -0.02" rpy="0 0 0"/>
+  </joint>
+  <!-- 3段目 -->
+  <link name="3rd_shelf">
+    <visual>
+      <origin xyz="0.0 0.0 0.0" rpy="0 0 0" />
+      <geometry>
+        <box size="0.95 0.454 0.0005" />
+      </geometry>
+      <material name="light_yellow">
+        <color rgba="01.0 1.0 0.7 1.0" />
+      </material>
+    </visual>
+    <collision>
+      <origin xyz="0.0 0.0 0.0" rpy="0 0 0" />
+      <geometry>
+        <box size="0.95 0.454 0.0005" />
+      </geometry>
+    </collision>
+  </link>
+  <joint name="3rd_shelf_joint" type="fixed">
+    <parent link="base_link"/>
+    <child link="3rd_shelf"/>
+    <origin xyz="0.0 -0.6 0.398" rpy="0 0 0"/>
+  </joint>
 </robot>

Commit message: 棚のurdfを修正

File: urdf/sciurus17.urdf.xacro (robot description, xacro)
@@ -224,5 +224,5 @@
     <parent link="base_link"/>
     <child link="first_shelf"/>
-    <origin xyz="0.0 -0.6 0.198" rpy="0 0 0"/>
+    <origin xyz="0.0 -0.6 -0.02" rpy="0 0 0"/>
   </joint>
   <!-- 2段目 -->
@@ -245,7 +245,7 @@
   </link>
   <joint name="2nd_shelf_joint" type="fixed">
-    <parent link="base_link"/>
+    <parent link="first_shelf"/>
     <child link="2nd_shelf"/>
-    <origin xyz="0.0 -0.6 -0.02" rpy="0 0 0"/>
+    <origin xyz="0.0 0.0 0.2" rpy="0 0 0"/>
   </joint>
   <!-- 3段目 -->
@@ -268,7 +268,7 @@
   </link>
   <joint name="3rd_shelf_joint" type="fixed">
-    <parent link="base_link"/>
+    <parent link="2nd_shelf"/>
     <child link="3rd_shelf"/>
-    <origin xyz="0.0 -0.6 0.398" rpy="0 0 0"/>
+    <origin xyz="0.0 0.0 0.2" rpy="0 0 0"/>
   </joint>
 </robot>

Commit message: 棚の位置を変更

File: urdf/sciurus17.urdf.xacro (robot description, xacro)
@@ -214,15 +214,15 @@
       </material>
     </visual>
-    <collision>
-      <origin xyz="0.0 0.0 0.0" rpy="0 0 0" />
-      <geometry>
-        <box size="0.95 0.454 0.0005" />
-      </geometry>
-    </collision>
+    <!-- <collision>
+      <origin xyz="0.0 0.0 0.0" rpy="0 0 0" />
+      <geometry>
+        <box size="0.95 0.454 0.0005" />
+      </geometry>
+    </collision> -->
   </link>
   <joint name="first_shelf_joint" type="fixed">
     <parent link="base_link"/>
     <child link="first_shelf"/>
-    <origin xyz="0.0 -0.6 -0.02" rpy="0 0 0"/>
+    <origin xyz="0.0 -0.45 -0.02" rpy="0 0 0"/>
   </joint>
   <!-- 2段目 -->
@@ -260,10 +260,10 @@
       </material>
     </visual>
-    <collision>
-      <origin xyz="0.0 0.0 0.0" rpy="0 0 0" />
-      <geometry>
-        <box size="0.95 0.454 0.0005" />
-      </geometry>
-    </collision>
+    <!-- <collision>
+      <origin xyz="0.0 0.0 0.0" rpy="0 0 0" />
+      <geometry>
+        <box size="0.95 0.454 0.0005" />
+      </geometry>
+    </collision> -->
   </link>
   <joint name="3rd_shelf_joint" type="fixed">
